File: board_1.0/bitraf_hydroponics.sch (KiCad schematic (older format))
At the start: 40 parts, among them P1 12V, P10 I2C_4, P11 BUZZ, P12 LDR, P13 TEMP_HUM, P14 PROGRAMMER, P15 SPI, P16 RADIO_433, P2 SWITCH_1, P3 SWITCH_2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

Commit message: o Renaming BUZZ to BUZZER now that it is visible on the PCB.
Parts:
- P11: value BUZZ -> BUZZER
Changed lines of the file:
@@
 P 7700 4400
 F 0 "P11" H 7700 4500 50  0000 C CNN
-F 1 "BUZZ" H 7700 4200 50  0000 C CNN
+F 1 "BUZZER" H 7700 4200 50  0000 C CNN
 F 2 "Bitraf:PhoenixContact_PTSM0,5_2-2,5-H_SMD" H 7700 4400 50  0001 C CNN
 F 3 "" H 7700 4400 50  0001 C CNN

Commit message: o Switching to new footprints for connectors. Moves everything around a little bit. o Adding some silk screen text to better indicate what goes where.
Connections:
- net +12V: now also P1.1 (Pin_1); no longer P1.2 (Pin_2)
- net GND: now also P1.2 (Pin_2); no longer P1.1 (Pin_1)
Changed lines of the file:
@@
 L Conn_01x02 P1
 U 1 1 57E46A8E
-P 1200 2400
-F 0 "P1" H 1200 2500 50  0000 C CNN
-F 1 "12V" H 1200 2200 50  0000 C CNN
-F 2 "Bitraf:PhoenixContact_PTSM0,5_2-2,5-H_SMD" H 1200 2400 50  0001 C CNN
-F 3 "" H 1200 2400 50  0001 C CNN
-	1    1200 2400
-	-1   0    0    1
+P 1200 2300
+F 0 "P1" H 1200 2400 50  0000 C CNN
+F 1 "12V" H 1200 2100 50  0000 C CNN
+F 2 "Bitraf:PhoenixContact_PTSM0,5_2-2,5-H_SMD" H 1200 2300 50  0001 C CNN
+F 3 "" H 1200 2300 50  0001 C CNN
+	1    1200 2300
+	-1   0    0    -1
 $EndComp
 $Comp

Commit message: o Adding mpn and other misc stuff. The forgotten commit.
Parts:
- C1: mpn (none) -> CL21B104MBCNNNC; voltage (none) -> 10V
- C2: mpn (none) -> GMK212BBJ106KG-T; req_voltage (none) -> 35V
- C3: mpn (none) -> GMK212BJ104KGHT; req_voltage (none) -> 35V; ta_ref 0.1u -> (none); ta_value (none) -> 0.1u
- C4: mpn (none) -> 08051A750JAT2A; voltage (none) -> 10V
- C5, C6: mpn (none) -> CL21A226MQCLQNC; voltage (none) -> 10V
- C7, C8: mpn (none) -> LMK212BJ475KD-T
- D1, D2, D3: digikey (none) -> 1655-1506-2-ND; mpn (none) -> S1MTR
- P1, P11, P12, P2, P3, P4: mpn (none) -> 1702473
- P10, P7, P8, P9: mpn (none) -> 826926-4
- P13: mpn (none) -> 826926-3
- P14, R6: assembly (none) -> DNO
- P15: mpn (none) -> 826926-6
- P16: mpn (none) -> PPPC031LFBN-RC
- P5, P6: mpn (none) -> 826926-5
- Q1, Q2, Q3: mpn (none) -> DMN2041L-7
- R1, R2, R3: mpn (none) -> RC0805FR-0710KL
- R4: mpn (none) -> RC0805FR-07100KL
- R5: mpn (none) -> RC0805FR-0713K3L
- U2: mpn (none) -> AP2114H-3.3TRG1
Other:
- note added: "Capacitors are\nrated to 10V"
- note added: "Capacitors are\nrated to 35V"
- note added: "Normall not installed"
Changed lines of the file:
@@
 F 2 "TO_SOT_Packages_SMD:SOT-23" H 7600 1700 50  0001 C CNN
 F 3 "" H 7400 1600 50  0000 C CNN
+F 4 "DMN2041L-7" H 7400 1600 60  0001 C CNN "mpn"
 	1    7400 1600
 	1    0    0    -1
@@
 F 2 "Bitraf:PhoenixContact_PTSM0,5_2-2,5-H_SMD" H 7800 1000 50  0001 C CNN
 F 3 "" H 7800 1000 50  0001 C CNN
+F 4 "1702473" H 7800 1000 60  0001 C CNN "mpn"
 	1    7800 1000
 	1    0    0    -1
@@
 F 2 "Diodes_SMD:D_SMA_Handsoldering" H 7300 1050 50  0001 C CNN
 F 3 "http://www.smc-diodes.com/propdf/S1A-S1M%20N0560%20REV.B.pdf" H 7300 1050 50  0001 C CNN
+F 4 "S1MTR" H 7300 1050 60  0001 C CNN "mpn"
+F 5 "1655-1506-2-ND" H 7300 1050 60  0001 C CNN "digikey"
 	1    7300 1050
 	0    1    1    0
@@
 F 2 "Resistors_SMD:R_0805" V 7030 1850 50  0001 C CNN
 F 3 "" H 7100 1850 50  0000 C CNN
+F 4 "RC0805FR-0710KL" V 7100 1850 60  0001 C CNN "mpn"
 	1    7100 1850
 	1    0    0    -1
@@
 F 2 "TO_SOT_Packages_SMD:SOT-23" H 9100 1700 50  0001 C CNN
 F 3 "" H 8900 1600 50  0000 C CNN
+F 4 "DMN2041L-7" H 8900 1600 60  0001 C CNN "mpn"
 	1    8900 1600
 	1    0    0    -1
@@
 F 2 "Bitraf:PhoenixContact_PTSM0,5_2-2,5-H_SMD" H 9300 1000 50  0001 C CNN
 F 3 "" H 9300 1000 50  0001 C CNN
+F 4 "1702473" H 9300 1000 60  0001 C CNN "mpn"
 	1    9300 1000
 	1    0    0    -1
@@
 F 2 "Resistors_SMD:R_0805" V 8530 1850 50  0001 C CNN
 F 3 "" H 8600 1850 50  0000 C CNN
+F 4 "RC0805FR-0710KL" V 8600 1850 60  0001 C CNN "mpn"
 	1    8600 1850
 	1    0    0    -1
@@
 F 2 "TO_SOT_Packages_SMD:SOT-23" H 10600 1700 50  0001 C CNN
 F 3 "" H 10400 1600 50  0000 C CNN
+F 4 "DMN2041L-7" H 10400 1600 60  0001 C CNN "mpn"
 	1    10400 1600
 	1    0    0    -1
@@
 F 2 "Bitraf:PhoenixContact_PTSM0,5_2-2,5-H_SMD" H 10800 1000 50  0001 C CNN
 F 3 "" H 10800 1000 50  0001 C CNN
+F 4 "1702473" H 10800 1000 60  0001 C CNN "mpn"
 	1    10800 1000
 	1    0    0    -1
@@
 F 2 "Resistors_SMD:R_0805" V 10030 1850 50  0001 C CNN
 F 3 "" H 10100 1850 50  0000 C CNN
+F 4 "RC0805FR-0710KL" V 10100 1850 60  0001 C CNN "mpn"
 	1    10100 1850
 	1    0    0    -1
@@
 F 2 "Socket_Strips:Socket_Strip_Straight_1x03_Pitch2.54mm" H 6500 7200 50  0001 C CNN
 F 3 "" H 6500 7200 50  0001 C CNN
+F 4 "PPPC031LFBN-RC" H 6500 7200 60  0001 C CNN "mpn"
 	1    6500 7200
 	1    0    0    -1
@@
 F 2 "Pin_Headers:Pin_Header_Straight_1x04_Pitch2.54mm" H 7700 3300 50  0001 C CNN
 F 3 "" H 7700 3300 50  0001 C CNN
+F 4 "826926-5" H 7700 3300 60  0001 C CNN "mpn"
 	1    7700 3300
 	1    0    0    -1
@@
 F 2 "Pin_Headers:Pin_Header_Straight_1x05_Pitch2.54mm" H 9400 3400 50  0001 C CNN
 F 3 "" H 9400 3400 50  0001 C CNN
+F 4 "826926-5" H 9400 3400 60  0001 C CNN "mpn"
 	1    9400 3400
 	1    0    0    -1
@@
 F 2 "Capacitors_SMD:C_0805" H 2138 2400 50  0001 C CNN
 F 3 "" H 2100 2550 50  0000 C CNN
-F 4 "0.1u" H 2100 2550 60  0001 C CNN "ta_ref"
+F 4 "0.1u" H 2100 2550 60  0001 C CNN "ta_value"
+F 5 "35V" H 2200 2350 60  0001 C CNN "req_voltage"
+F 6 "GMK212BJ104KGHT" H 2100 2550 60  0001 C CNN "mpn"
 	1    2100 2550
 	1    0    0    -1
@@
 F 3 "" H 5500 2550 50  0000 C CNN
 F 4 "C4" H 5500 2550 60  0001 C CNN "ta_ref"
+F 5 "10V" H 5500 2550 60  0001 C CNN "voltage"
+F 6 "CL21A226MQCLQNC" H 5500 2550 60  0001 C CNN "mpn"
 	1    5500 2550
 	1    0    0    -1
@@
 F 3 "" H 1800 2550 50  0000 C CNN
 F 4 "C1" H 1800 2550 60  0001 C CNN "ta_ref"
+F 5 "35V" H 1900 2350 60  0001 C CNN "req_voltage"
+F 6 "GMK212BBJ106KG-T" H 1800 2550 60  0001 C CNN "mpn"
 	1    1800 2550
 	1    0    0    -1
@@
 F 3 "" H 5800 2550 50  0000 C CNN
 F 4 "C5" H 5800 2550 60  0001 C CNN "ta_ref"
+F 5 "10V" H 5800 2550 60  0001 C CNN "voltage"
+F 6 "CL21A226MQCLQNC" H 5800 2550 60  0001 C CNN "mpn"
 	1    5800 2550
 	1    0    0    -1
@@
 F 2 "Bitraf:PhoenixContact_PTSM0,5_2-2,5-H_SMD" H 1200 2300 50  0001 C CNN
 F 3 "" H 1200 2300 50  0001 C CNN
+F 4 "1702473" H 1200 2300 60  0001 C CNN "mpn"
 	1    1200 2300
 	-1   0    0    -1
@@
 F 2 "Bitraf:PhoenixContact_PTSM0,5_2-2,5-H_SMD" H 7700 4400 50  0001 C CNN
 F 3 "" H 7700 4400 50  0001 C CNN
+F 4 "1702473" H 7700 4400 60  0001 C CNN "mpn"
 	1    7700 4400
 	1    0    0    -1
@@
 F 2 "Bitraf:PhoenixContact_PTSM0,5_2-2,5-H_SMD" H 9350 4650 50  0001 C CNN
 F 3 "" H 9350 4650 50  0001 C CNN
+F 4 "1702473" H 9350 4650 60  0001 C CNN "mpn"
 	1    9350 4650
 	1    0    0    -1
@@
 F 2 "Resistors_THT:R_Axial_DIN0207_L6.3mm_D2.5mm_P10.16mm_Horizontal" V 8980 5000 50  0001 C CNN
 F 3 "" H 9050 5000 50  0000 C CNN
+F 4 "DNO" V 8950 5000 60  0000 C CNN "assembly"
 	1    9050 5000
 	1    0    0    -1
@@
 F 2 "Pin_Headers:Pin_Header_Straight_1x03_Pitch2.54mm" H 7600 5600 50  0001 C CNN
 F 3 "" H 7600 5600 50  0001 C CNN
+F 4 "826926-3" H 7600 5600 60  0001 C CNN "mpn"
 	1    7600 5600
 	1    0    0    -1
@@
 F 2 "Pin_Headers:Pin_Header_Straight_1x04_Pitch2.54mm" H 10900 3500 50  0001 C CNN
 F 3 "" H 10900 3500 50  0001 C CNN
+F 4 "826926-4" H 10900 3500 60  0001 C CNN "mpn"
 	1    10900 3500
 	1    0    0    -1
@@
 F 2 "Pin_Headers:Pin_Header_Straight_1x04_Pitch2.54mm" H 10900 4100 50  0001 C CNN
 F 3 "" H 10900 4100 50  0001 C CNN
+F 4 "826926-4" H 10900 4100 60  0001 C CNN "mpn"
 	1    10900 4100
 	1    0    0    -1
@@
 F 2 "Pin_Headers:Pin_Header_Straight_1x04_Pitch2.54mm" H 10900 4700 50  0001 C CNN
 F 3 "" H 10900 4700 50  0001 C CNN
+F 4 "826926-4" H 10900 4700 60  0001 C CNN "mpn"
 	1    10900 4700
 	1    0    0    -1
@@
 F 2 "Pin_Headers:Pin_Header_Straight_1x04_Pitch2.54mm" H 10900 5300 50  0001 C CNN
 F 3 "" H 10900 5300 50  0001 C CNN
+F 4 "826926-4" H 10900 5300 60  0001 C CNN "mpn"
 	1    10900 5300
 	1    0    0    -1
@@
 F 5 "TPS54202DDCT" H 3100 2300 60  0001 C CNN "mpn"
 F 6 "2A" H 2800 3000 60  0000 C CNN "Iout"
-F 7 "5V" H 3000 3000 60  0000 C CNN "Vout"
+F 7 "5V" H 3350 3000 60  0000 C CNN "Vout"
 	1    3100 2300
 	1    0    0    -1
@@
 F 3 "" H 5000 2550 50  0000 C CNN
 F 4 "R2" V 5000 2550 60  0001 C CNN "ta_ref"
+F 5 "RC0805FR-07100KL" V 5000 2550 60  0001 C CNN "mpn"
 	1    5000 2550
 	1    0    0    -1
@@
 F 3 "" H 4000 2050 50  0000 C CNN
 F 4 "C3" H 4000 2050 60  0001 C CNN "ta_ref"
+F 5 "10V" H 4000 2050 60  0001 C CNN "voltage"
+F 6 "CL21B104MBCNNNC" H 4000 2050 60  0001 C CNN "mpn"
 	1    4000 2050
 	1    0    0    -1
@@
 F 2 "Pin_Headers:Pin_Header_Straight_1x06_Pitch2.54mm" H 5100 7100 50  0001 C CNN
 F 3 "" H 5100 7100 50  0001 C CNN
+F 4 "826926-6" H 5100 7100 60  0001 C CNN "mpn"
 	1    5100 7100
 	1    0    0    -1
@@
 F 3 "" H 5000 3050 50  0000 C CNN
 F 4 "R3" V 5000 3050 60  0001 C CNN "ta_ref"
+F 5 "RC0805FR-0713K3L" V 5000 3050 60  0001 C CNN "mpn"
 	1    5000 3050
 	1    0    0    -1
@@
 F 3 "" H 4700 2550 50  0000 C CNN
 F 4 "C6" H 4700 2550 60  0001 C CNN "ta_ref"
+F 5 "10V" H 4700 2550 60  0001 C CNN "voltage"
+F 6 "08051A750JAT2A" H 4700 2550 60  0001 C CNN "mpn"
 	1    4700 2550
 	1    0    0    -1
@@
 F 2 "TO_SOT_Packages_SMD:SOT-223" H 1700 4500 60  0001 C CNN
 F 3 "" H 1700 4500 60  0001 C CNN
-F 4 "1A" H 1000 3200 60  0001 L BNN "Iout"
+F 4 "1A" H 1900 4800 60  0000 L BNN "Iout"
+F 5 "AP2114H-3.3TRG1" H 1700 4500 60  0001 C CNN "mpn"
 	1    1700 4500
 	1    0    0    -1
@@
 F 2 "Capacitors_SMD:C_0805" H 838 4500 50  0001 C CNN
 F 3 "" H 800 4650 50  0001 C CNN
+F 4 "LMK212BJ475KD-T" H 800 4650 60  0001 C CNN "mpn"
 	1    800  4650
 	1    0    0    -1
@@
 F 2 "Capacitors_SMD:C_0805" H 2838 4500 50  0001 C CNN
 F 3 "" H 2800 4650 50  0001 C CNN
+F 4 "LMK212BJ475KD-T" H 2800 4650 60  0001 C CNN "mpn"
 	1    2800 4650
 	1    0    0    -1
@@
 F 2 "Pin_Headers:Pin_Header_Straight_1x06_Pitch2.54mm" H 3400 7100 50  0001 C CNN
 F 3 "" H 3400 7100 50  0001 C CNN
+F 4 "DNO" V 3600 6850 60  0000 C CNN "assembly"
 	1    3400 7100
 	1    0    0    -1
@@
 F 2 "Diodes_SMD:D_SMA_Handsoldering" H 8800 1050 50  0001 C CNN
 F 3 "http://www.smc-diodes.com/propdf/S1A-S1M%20N0560%20REV.B.pdf" H 8800 1050 50  0001 C CNN
+F 4 "S1MTR" H 8800 1050 60  0001 C CNN "mpn"
+F 5 "1655-1506-2-ND" H 8800 1050 60  0001 C CNN "digikey"
 	1    8800 1050
 	0    1    1    0
@@
 F 2 "Diodes_SMD:D_SMA_Handsoldering" H 10300 1050 50  0001 C CNN
 F 3 "http://www.smc-diodes.com/propdf/S1A-S1M%20N0560%20REV.B.pdf" H 10300 1050 50  0001 C CNN
+F 4 "S1MTR" H 10300 1050 60  0001 C CNN "mpn"
+F 5 "1655-1506-2-ND" H 10300 1050 60  0001 C CNN "digikey"
 	1    10300 1050
 	0    1    1    0
 $EndComp
 Connection ~ 5000 2300
+Text Notes 1800 2200 0    40   ~ 0
+Capacitors are\nrated to 35V
+Text Notes 4500 2200 0    40   ~ 0
+Capacitors are\nrated to 10V
+Text Notes 3750 7300 1    40   ~ 0
+Normall not installed
 $EndSCHEMATC

Commit message: Added pullups and jumper header fro programming. Still need to tweak the mosfets, but need expert help
Parts:
- added J1: PRG_JMP, Pin_Headers:Pin_Header_Straight_1x02_Pitch2.54mm, symbol Conn_01x02
- added R7: 8.2k, Resistors_SMD:R_0805, symbol R
Connections:
- net CH_PD is gone; now on net +3V3: P14.2 (Pin_2), U3.3 (CH_PD)
- net +3V3: now also R7.1
- net TEMP_HUM: now also R7.2
- net ROT_0 renamed PRG
- net PRG: now also J1.2 (Pin_2)
- new net RESET: J1.1 (Pin_1)
Other:
- note added: "Jumper for programming"

Commit message: This should go in it's own branch/folder. Revert "Added pullups and jumper header fro programming. Still need to tweak the mosfets, but need expert help"
This reverts commit b0ba335143d29f2dde67b78845eb19ede0b5a3d2.
Parts:
- removed J1: PRG_JMP, Pin_Headers:Pin_Header_Straight_1x02_Pitch2.54mm, symbol Conn_01x02
- removed R7: 8.2k, Resistors_SMD:R_0805, symbol R
Connections:
- net +3V3: no longer P14.2 (Pin_2), U3.3 (CH_PD)
- net PRG renamed ROT_0
- new net CH_PD: P14.2 (Pin_2), U3.3 (CH_PD)
Other:
- note removed: "Jumper for programming"
